File: hardware/nanoleaf_shapes.kicad_sch (KiCad schematic)
At the start: 42 parts, among them J1 Conn_01x03, J2 Conn_01x03, SW1 RESET, SW2 BOOT, U1 TPS54360DDAR, U2 WT0132C6-S5, U3 74LVC1G125GV_C52140413, U4 74LVC1G125GV_C52140413

Commit message: Rev B hardware: replaces rev A, not yet verified
Rev B clips onto a panel like the stock controller instead of connecting
through a cut flex linker, and fixes the rev A issues listed in the README.
It replaces rev A in hardware/.

NOT VERIFIED. No rev B board has been built or powered up. Boards are on
order. What has been checked is DRC (0 errors, 0 unconnected items), ground
continuity, a 3D fit check of the enclosure against the KiCad component
models, and the fabrication files against the board they came from. None of
that proves the circuit works. Rev A, which is built and working, stays in
the history at the previous commit.

Also added:

- mechanical/ builds the enclosure from the board itself. export_parts.py
  dumps the geometry out of KiCad, enclosure.py turns it into a tray, a lid
  and three separate button caps, and make_fab_files.py writes the BOM and
  placement files. case_v1_working/ keeps the previous enclosure as a
  fallback, with the sources and parts.json that produced it.
- fab/pcbway/ holds the gerbers, drill files, BOM and centroid file.
- render/ holds three KiCad 3D renders, shown in the README.

The JLCPCB fabrication files are deliberately not published. PCBWay are
sponsoring this board, and that file set also carries corrections that only
make sense against JLCPCB's own library.

Co-Authored-By: Claude Opus 5 <noreply@anthropic.com>
Parts:
- removed J2: Conn_01x03, Connector_PinHeader_2.54mm:PinHeader_1x03_P2.54mm_Vertical, symbol Connector_Generic:Conn_01x03
- added C22, C23, C24, C26: 100nF 16V, easyeda2kicad:C0402, symbol Device:C
- added D3: SMAJ48A, Diode_SMD:D_SMA, symbol Diode:SMAJ48A
- added D4: LED, LED_SMD:LED_0603_1608Metric, symbol Device:LED
- added D5: 100V/2A Schottky, Diode_SMD:D_SMA, symbol Device:D
- added J3: USB_C_Receptacle_USB2.0_16P, Connector_USB:USB_C_Receptacle_HRO_TYPE-C-31-M-12, symbol Connector:USB_C_Receptacle_USB2.0_16P
- added Q1, Q2: MMBT3904, Package_TO_SOT_SMD:SOT-23, symbol Transistor_BJT:MMBT3904
- added R11, R12: 5.1k, easyeda2kicad:R0402, symbol Device:R
- added R13, R14, R16: 10k, easyeda2kicad:R0402, symbol Device:R
- added R15: 100k, easyeda2kicad:R0402, symbol Device:R
- added R17: 1k, easyeda2kicad:R0402, symbol Device:R
- added SW3, SW4, SW6: USER BUTTON, Button_Switch_SMD:SW_Push_1P1T_XKB_TS-1187A, symbol easyeda2kicad:TS-1088-AR02016
- added U5: CH340C, Package_SO:SOIC-16_3.9x9.9mm_P1.27mm, symbol Interface_USB:CH340C
- added U6: USBLC6-2SC6, Package_TO_SOT_SMD:SOT-23-6, symbol Power_Protection:USBLC6-2SC6
- C11: value 22uF 100V -> 2.2uF 100V; footprint easyeda2kicad:CAP-SMD_BD6.3-L6.6-W6.6-FD-1 -> easyeda2kicad:C1210; JLCPCB C47023097 -> C5449052
- J1: footprint Connector_PinHeader_2.54mm:PinHeader_1x03_P2.54mm_Vertical -> nanoleaf:Nanoleaf_Linker_Pads; now left out of the parts list
- SW1, SW2: footprint easyeda2kicad:SW-SMD_L3.9-W3.0-P4.45 -> Button_Switch_SMD:SW_SPST_TS-1088-xR020; JLCPCB (none) -> C720477
- U1: JLCPCB (none) -> C44377
- U3, U4: JLCPCB (none) -> C52140413
Connections:
- net 3V3: now also C22.1, R15.1, R16.1, U5.16 (VCC), U5.4 (V3)
- net 42V: now also D3.1 (A1), D5.1 (K)
- net COM: now also R15.2
- net GND: now also C22.2, C23.2, C24.2, C26.2, D3.2 (A2), D4.1 (K), J3.A1 (GND), J3.A12 (GND), J3.B1 (GND), J3.B12 (GND), J3.SH (SHIELD), R11.2, R12.2, SW3.2, SW4.2, SW6.2, U5.1 (GND), U6.2 (GND)
- net RX0: now also U5.2 (TXD)
- net TX0: now also U5.3 (RXD)
- net BTN_PWR: now reaches U2.1 (GPIO0)
- net BTN_PWR: now also C23.1, SW3.1
- net at U2.11 (GPIO8): now also R16.2
- net BOOT: now reaches SW2.1, U2.12 (GPIO9)
- net BOOT: now also Q1.3 (C)
- net at U2.18 (GPIO19): now also R17.1
- net BTN_UP: now reaches U2.2 (GPIO1)
- net BTN_UP: now also C24.1, SW4.1
- net BTN_DN: now reaches U2.20 (GPIO21)
- net BTN_DN: now also C26.1, SW6.1
- new net: D4.2 (A), R17.2
- new net: Q2.2 (E), R13.1, U5.13 (~{DTR})
- new net: Q1.1 (B), R13.2
- new net: Q1.2 (E), R14.1, U5.14 (~{RTS})
- new net: J3.A5 (CC1), R11.1
- new net: J3.B5 (CC2), R12.1
- new net: Q2.1 (B), R14.2
- new net EN: Q2.3 (C)
- new net USB_DN: J3.A7 (D-), J3.B7 (D-), U5.6 (UD-), U6.3 (I/O2), U6.4 (I/O2)
- new net USB_DP: J3.A6 (D+), J3.B6 (D+), U5.5 (UD+), U6.1 (I/O1), U6.6 (I/O1)
- new net USB_VBUS: D5.2 (A), J3.A4 (VBUS), J3.A9 (VBUS), J3.B4 (VBUS), J3.B9 (VBUS), U6.5 (VBUS)
- no-connect marks 14 -> 17
Other:
- moved on the sheet: C17, C18, C19, D2, R1, R10, R6, R7, SW2, U3, U4
